File: StripeV02.sch (KiCad schematic (older format))
At the start: 28 parts, among them J1 USB_SOCKET, K1 CONN_3, P3 CONN_1, P4 CONN_1, P5 CONN_1, U1 CARAMBOLA

Commit message: RFM12B hookup
Parts:
- removed ISP: CONN_3X2, symbol CONN_3X2
- added CON?: AVR-ISP-6, AVR-ISP-6, symbol AVR-ISP-6
- C1: value 22u -> 22µ
- C?: value C -> 1µ
- R? (x2): value R -> 10K
Connections:
- wire segments 70 -> 91
Other:
- note added: "Test points"
- moved on the sheet: C?, IC?, P3, P4, P5, R?
Changed lines of the file:
@@
-EESchema Schematic File Version 2  date Tue 17 Apr 2012 11:18:13 PM CEST
+EESchema Schematic File Version 2  date Wed 18 Apr 2012 12:04:37 AM CEST
 LIBS:power
 LIBS:device
@@
 Text Label 4850 5250 0    60   ~ 0
 VSW
-Text Label 4700 1300 0    60   ~ 0
+Text Label 10400 6850 0    60   ~ 0
 3.3VD
-Text Label 4700 1100 0    60   ~ 0
+Text Label 10400 6650 0    60   ~ 0
 5VD
-Text Label 4700 900  0    60   ~ 0
+Text Label 10400 6450 0    60   ~ 0
 GND
 $Comp
 L CONN_1 P5
 U 1 1 4F3FB113
-P 4850 1300
-F 0 "P5" H 4930 1300 40  0000 L CNN
-F 1 "CONN_1" H 4850 1355 30  0001 C CNN
-	1    4850 1300
+P 10550 6850
+F 0 "P5" H 10630 6850 40  0000 L CNN
+F 1 "CONN_1" H 10550 6905 30  0001 C CNN
+	1    10550 6850
 	1    0    0    -1
 $EndComp
@@
 L CONN_1 P4
 U 1 1 4F3FB104
-P 4850 1100
-F 0 "P4" H 4930 1100 40  0000 L CNN
-F 1 "CONN_1" H 4850 1155 30  0001 C CNN
-	1    4850 1100
+P 10550 6650
+F 0 "P4" H 10630 6650 40  0000 L CNN
+F 1 "CONN_1" H 10550 6705 30  0001 C CNN
+	1    10550 6650
 	1    0    0    -1
 $EndComp
@@
 L CONN_1 P3
 U 1 1 4F3FB0F5
-P 4850 900
-F 0 "P3" H 4930 900 40  0000 L CNN
-F 1 "CONN_1" H 4850 955 30  0001 C CNN
-	1    4850 900
+P 10550 6450
+F 0 "P3" H 10630 6450 40  0000 L CNN
+F 1 "CONN_1" H 10550 6505 30  0001 C CNN
+	1    10550 6450
 	1    0    0    -1
 $EndComp
@@
 P 2950 5600
 F 0 "C1" H 3000 5700 50  0000 L CNN
-F 1 "22u" H 3000 5500 50  0000 L CNN
+F 1 "22µ" H 3000 5500 50  0000 L CNN
 	1    2950 5600
 	1    0    0    -1
@@
 F 2 "DIP14" H 1450 1250 60  0001 C CNN
 	1    2150 2000
-	1    0    0    1
+	1    0    0    -1
 $EndComp
 $Comp
 L C C?
 U 1 1 4F8DDAB4
-P 1050 2000
-F 0 "C?" H 1100 2100 50  0000 L CNN
-F 1 "C" H 1100 1900 50  0000 L CNN
-	1    1050 2000
+P 950 1950
+F 0 "C?" H 1000 2050 50  0000 L CNN
+F 1 "1µ" H 1000 1850 50  0000 L CNN
+	1    950  1950
 	1    0    0    -1
 $EndComp
@@
 L R R?
 U 1 1 4F8DDAC3
-P 3400 1050
-F 0 "R?" V 3480 1050 50  0000 C CNN
-F 1 "R" V 3400 1050 50  0000 C CNN
-	1    3400 1050
-	1    0    0    -1
+P 3950 2400
+F 0 "R?" V 4030 2400 50  0000 C CNN
+F 1 "10K" V 3950 2400 50  0000 C CNN
+	1    3950 2400
+	0    -1   -1   0
 $EndComp
 $Comp
 L R R?
 U 1 1 4F8DDAD2
-P 3650 1050
-F 0 "R?" V 3750 1050 50  0000 C CNN
-F 1 "R" V 3650 1050 50  0000 C CNN
-	1    3650 1050
-	1    0    0    -1
-$EndComp
-$Comp
-L CONN_3X2 ISP
-U 1 1 4F8DDB4F
-P 2250 3200
-F 0 "ISP" H 2250 3450 50  0000 C CNN
-F 1 "CONN_3X2" V 2250 3250 40  0000 C CNN
-	1    2250 3200
-	1    0    0    -1
+P 3950 2600
+F 0 "R?" V 4050 2600 50  0000 C CNN
+F 1 "10K" V 3950 2600 50  0000 C CNN
+	1    3950 2600
+	0    -1   -1   0
 $EndComp
 $Comp
@@
 	1    0    0    -1
 $EndComp
+$Comp
+L RFM12 IC?
+U 1 1 4F8DE358
+P 4200 3350
+F 0 "IC?" H 3900 2900 60  0000 C CNN
+F 1 "RFM12" H 4200 3350 60  0000 C CNN
+	1    4200 3350
+	1    0    0    -1
+$EndComp
+$Comp
+L AVR-ISP-6 CON?
+U 1 1 4F8DE92F
+P 2200 3400
+F 0 "CON?" H 2120 3640 50  0000 C CNN
+F 1 "AVR-ISP-6" H 1960 3170 50  0000 L BNN
+F 2 "AVR-ISP-6" V 1680 3440 50  0001 C CNN
+	1    2200 3400
+	1    0    0    -1
+$EndComp
+Text Notes 10350 6200 0    60   ~ 0
+Test points
 Wire Wire Line
 	8700 3150 8800 3150
@@
 Wire Wire Line
 	1700 6300 1700 6450
-$Comp
-L RFM12 IC?
-U 1 1 4F8DE358
-P 5100 3100
-F 0 "IC?" H 4600 2400 60  0000 C CNN
-F 1 "RFM12" H 5100 3100 60  0000 C CNN
-	1    5100 3100
-	1    0    0    -1
-$EndComp
+Wire Wire Line
+	3200 2500 3350 2500
+Wire Wire Line
+	3350 2500 3350 3600
+Wire Wire Line
+	3350 3600 3650 3600
+Wire Wire Line
+	3200 2000 3400 2000
+Wire Wire Line
+	3400 2000 3400 3400
+Wire Wire Line
+	3400 3400 3650 3400
+Wire Wire Line
+	3200 1900 3450 1900
+Wire Wire Line
+	3450 1900 3450 3300
+Wire Wire Line
+	3450 3300 3650 3300
+Wire Wire Line
+	3200 1800 3500 1800
+Wire Wire Line
+	3500 1800 3500 3200
+Wire Wire Line
+	3500 3200 3650 3200
+Wire Wire Line
+	3650 3100 3550 3100
+Wire Wire Line
+	3550 3100 3550 2400
+Wire Wire Line
+	3200 2400 3700 2400
+Wire Wire Line
+	4200 2400 4200 2800
+Connection ~ 4200 2600
+Connection ~ 4200 2600
+Connection ~ 3550 2400
+Wire Wire Line
+	3200 2600 3700 2600
+Wire Wire Line
+	950  2150 950  2600
+Wire Wire Line
+	950  2600 1100 2600
+Wire Wire Line
+	1100 1400 950  1400
+Wire Wire Line
+	950  1400 950  1750
 $EndSCHEMATC

Commit message: Added 6PIN headers and minor cleanup
Parts:
- removed CON?: AVR-ISP-6, AVR-ISP-6, symbol AVR-ISP-6
- added AVR1: CONN_3X2, symbol CONN_3X2
- added P1: CONN_1, symbol CONN_1
- added P2: UART1, symbol CONN_6
- added P6: UART2, symbol CONN_6
- added P7, P8: I2C_PLUG, symbol CONN_6
- C2, C3: value 22u -> 22µ
- C7: value 100uF -> 100µ
- L1: value INDUCTOR -> 4R7
- gave numbers to parts that had none: 5
Connections:
- net labels added: AGND, PGND, RX2, TX2
- net labels removed: RX, TX
- wire segments 91 -> 114
- no-connect marks 0 -> 1
Other:
- note removed: "2 x 10K parallel instead of 1 x 5K"
- note removed: "3x10K in series instead of 1x30K"
- moved on the sheet: C1, C4, C5, C7, DC1, K1, L1, L2, L3, R1, R5, R6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
